Commit message: sim: define sensor colors in gazebo

File: robot_description/urdf/robot.gazebo.xacro (robot description, xacro)
@@ -27,4 +27,10 @@
     <xacro:caster_gazebo name="front_caster"/>
     <xacro:caster_gazebo name="rear_caster"/>
+    <gazebo reference="camera_link">
+        <material>Gazebo/Green</material>
+    </gazebo>
+    <gazebo reference="laser_link">
+        <material>Gazebo/Black</material>
+    </gazebo>
     <gazebo>
         <plugin name="gazebo_ros_control" filename="libgazebo_ros_control.so">

Commit message: sim: add camera plugin

File: robot_description/urdf/robot.gazebo.xacro (robot description, xacro)
@@ -27,7 +27,51 @@
     <xacro:caster_gazebo name="front_caster"/>
     <xacro:caster_gazebo name="rear_caster"/>
+    <!-- camera -->
     <gazebo reference="camera_link">
         <material>Gazebo/Green</material>
     </gazebo>
+    <gazebo reference="camera_link">
+        <sensor type="camera" name="camera">
+            <!-- 60 fps in sensors_base.launch -->
+            <update_rate>30.0</update_rate>
+            <camera name="head">
+                <horizontal_fov>${radians(62.2)}</horizontal_fov>
+                <image>
+                    <!-- img resolution from sensors_base.launch -->
+                    <width>1024</width>
+                    <height>576</height>
+                    <format>R8G8B8</format>
+                </image>
+                <clip>
+                    <near>0.02</near>
+                    <far>300</far>
+                </clip>
+                <noise>
+                    <type>gaussian</type>
+                    <!-- Noise is sampled independently per pixel on each frame.
+                         That pixel's noise value is added to each of its color
+                         channels, which at that point lie in the range [0,1]. -->
+                    <mean>0.0</mean>
+                    <stddev>0.007</stddev>
+                </noise>
+            </camera>
+            <plugin name="camera_controller" filename="libgazebo_ros_camera.so">
+                <alwaysOn>true</alwaysOn>
+                <updateRate>0.0</updateRate>
+                <robotNamespace>/</robotNamespace>
+                <cameraName>camera</cameraName>
+                <imageTopicName>image_raw</imageTopicName>
+                <cameraInfoTopicName>camera_info</cameraInfoTopicName>
+                <frameName>camera_link</frameName>
+                <hackBaseline>0.07</hackBaseline>
+                <distortionK1>0.0</distortionK1>
+                <distortionK2>0.0</distortionK2>
+                <distortionK3>0.0</distortionK3>
+                <distortionT1>0.0</distortionT1>
+                <distortionT2>0.0</distortionT2>
+            </plugin>
+        </sensor>
+    </gazebo>
+    <!-- laser -->
     <gazebo reference="laser_link">
         <material>Gazebo/Black</material>

File: robot_description/urdf/robot.urdf.xacro (robot description, xacro)
@@ -120,14 +120,14 @@
         <visual>
             <geometry>
-                <box size="${camera_length} ${camera_width} ${camera_thickness}"/>
+                <box size="${camera_thickness} ${camera_width} ${camera_length}"/>
             </geometry>
-            <origin xyz="${-camera_x_offset} 0 0"/>
+            <origin xyz="0 0 ${camera_x_offset}"/>
             <material name="green"/>
         </visual>
         <collision>
             <geometry>
-                <box size="${camera_length} ${camera_width} ${camera_thickness}"/>
+                <box size="${camera_thickness} ${camera_width} ${camera_length}"/>
             </geometry>
-            <origin xyz="${-camera_x_offset} 0 0"/>
+            <origin xyz="0 0 ${camera_x_offset}"/>
         </collision>
         <inertial>
@@ -135,5 +135,5 @@
             <!-- inertia tensor approximation using cuboid -->
             <inertia ixx="${1.02979e-5}" ixy="0" ixz="0" iyy="${1.1178e-5}" iyz="0" izz="${1.8911e-5}"/>
-            <origin xyz="${-camera_x_offset} 0 0"/>
+            <origin xyz="0 0 ${camera_x_offset}"/>
         </inertial>
     </link>
@@ -142,6 +142,6 @@
         <child link="camera_link"/>
         <origin xyz="${0.0602+camera_thickness/2} 0 ${base_height/2+0.0025+camera_sensor_x}"
-                rpy="0 ${pi/2} 0"/>
-        <axis xyz="0 0 1"/>
+                rpy="0 0 0"/>
+        <axis xyz="1 0 0"/>
     </joint>
     <!-- laser -->
