Commit message: teleop: fix viz issues
- tf
- sensor feeds
- lidar backwards

File: robot_description/urdf/robot.urdf.xacro (robot description, xacro)
@@ -153,5 +153,6 @@
                 <mesh filename="package://robot_description/meshes/rplidar_main.STL"/>
             </geometry>
-            <origin xyz="${-laser_x_offset} 0 ${-laser_sensor_z}"/>
+            <origin xyz="${laser_x_offset} 0 ${-laser_sensor_z}"
+                    rpy="0 0 ${pi}"/>
             <material name="black"/>
         </visual>
@@ -174,5 +175,5 @@
         <child link="laser_link"/>
         <origin xyz="0 0 ${laser_z_offset}"
-                rpy="0 0 0"/>
+                rpy="0 0 ${pi}"/>
         <axis xyz="0 0 1"/>
     </joint>

Commit message: make casters continuous

File: robot_description/urdf/robot.urdf.xacro (robot description, xacro)
@@ -105,9 +105,10 @@
             </inertial>
         </link>
-        <joint name="${parent_name}_to_${name}_joint" type="fixed">
+        <joint name="${parent_name}_to_${name}_joint" type="continuous">
             <parent link="${parent_name}_link"/>
             <child link="${link_name}"/>
             <origin xyz="${reflect*wheelbase_length/2} 0 -${caster_z_offset}"/>
             <dynamics friction="0"/>
+            <axis xyz="0 1 0"/>
         </joint>
     </xacro:macro>

Commit message: Revert "make casters continuous"
This reverts commit 3a9c5f69ece680231ff0b49033c50956b40bbc0b.

File: robot_description/urdf/robot.urdf.xacro (robot description, xacro)
@@ -105,10 +105,9 @@
             </inertial>
         </link>
-        <joint name="${parent_name}_to_${name}_joint" type="continuous">
+        <joint name="${parent_name}_to_${name}_joint" type="fixed">
             <parent link="${parent_name}_link"/>
             <child link="${link_name}"/>
             <origin xyz="${reflect*wheelbase_length/2} 0 -${caster_z_offset}"/>
             <dynamics friction="0"/>
-            <axis xyz="0 1 0"/>
         </joint>
     </xacro:macro>
